File: pcb/pcb.kicad_pcb (KiCad board)
At the start: 2 copper layers, 60 x 60 mm, 13 parts, among them SW2 SW_Push

Commit message: 5.9
Parts:
- moved BZ3 3.76 mm to (143.4, 80.0)
- moved ? 1.45 mm to (117.9, 72.7)
- moved U2 1.28 mm to (140.5, 82.2)
- moved ? 0.48 mm to (99.8, 85.8)
Routing:
- net +3.3V: track 142.1 -> 152.5 mm
- net Net-(U1-A2): track 24.2 -> 25.9 mm
- net Net-(BZ3-+): track 37.8 -> 36.1 mm
- net Net-(U1-11): track 9.26 -> 10.5 mm
- net Net-(U1-10): track 13.9 -> 15.2 mm
- net Net-(U1-A1): track 22.3 -> 23.6 mm
- net Net-(U4-GND): track 37.3 -> 36.1 mm
