File: pcb/_autosave-pcb.kicad_pcb (KiCad board)
At the start: 2 copper layers, 60 x 60 mm, 13 parts, among them SW2 SW_Push

Commit message: 5.10
Parts:
- moved BZ3 3.66 mm to (143.4, 80.0)
Routing:
- net GND: track 104.7 -> 103.1 mm
- net Net-(BZ3-+): track 37.6 -> 36.1 mm
Changed lines of the file:
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@@
 	(footprint "Buzzer_Beeper:Buzzer_12x9.5RM7.6"
 		(layer "F.Cu")
-		(at 143.4084 76.3016)
+		(at 143.4084 79.9592)
 		(descr "Generic Buzzer, D12mm height 9.5mm with RM7.6mm")
 		(tags "buzzer")
@@
 	)
 	(segment
-		(start 151.0084 76.3116)
-		(end 151.0084 76.3016)
-		(width 0.508)
-		(layer "F.Cu")
-		(net 1)
-	)
-	(segment
 		(start 113.9444 85.8774)
 		(end 113.9444 85.1916)
@@
 	)
 	(segment
-		(start 137.16 90.16)
-		(end 151.0084 76.3116)
-		(width 0.508)
-		(layer "F.Cu")
-		(net 1)
-	)
-	(segment
 		(start 123.7996 83.1596)
 		(end 129.54 88.9)
@@
 	)
 	(segment
+		(start 147.3608 79.9592)
+		(end 151.0084 79.9592)
+		(width 0.508)
+		(layer "F.Cu")
+		(net 1)
+	)
+	(segment
+		(start 137.16 91.44)
+		(end 137.16 90.16)
+		(width 0.508)
+		(layer "F.Cu")
+		(net 1)
+	)
+	(segment
 		(start 142.0876 101.0412)
 		(end 137.16 96.1136)
@@
 	)
 	(segment
-		(start 137.16 91.44)
-		(end 137.16 90.16)
+		(start 137.16 90.16)
+		(end 147.3608 79.9592)
 		(width 0.508)
 		(layer "F.Cu")
@@
 	)
 	(segment
-		(start 143.4084 76.3016)
-		(end 143.4084 76.3116)
+		(start 143.4084 79.9592)
+		(end 139.7608 79.9592)
 		(width 0.381)
 		(layer "F.Cu")
@@
 	)
 	(segment
-		(start 130.9605 100.2844)
-		(end 124.9426 106.3023)
+		(start 139.7608 79.9592)
+		(end 130.9605 88.7595)
 		(width 0.381)
 		(layer "F.Cu")
@@
 	)
 	(segment
-		(start 143.4084 76.3116)
-		(end 130.9605 88.7595)
+		(start 130.9605 100.2844)
+		(end 124.9426 106.3023)
 		(width 0.381)
 		(layer "F.Cu")
